Commit message: add holder
change robot orientation and add right holder

File: urdf_description/urdf/first.urdf (robot description, URDF)
Before this commit: robot myfirst, 7 links, 6 joints
Links:
- added link right_front_holder; visual box size=0.02 0.08 0.01
Joints:
- added joint base_to_right_front_holder: type fixed, parent base_link, child right_front_holder, origin xyz=0 0 0
- joint base_to_right_front_caster_wheel: parent base_link -> right_front_holder

Commit message: change joints
changing joint origins and observing differences

File: urdf_description/urdf/first.urdf (robot description, URDF)
Before this commit: robot myfirst, 8 links, 7 joints
Joints:
- joint base_to_left_back_caster_wheel: origin xyz=0 0 0 -> xyz=-0.375 0.170 0
- joint base_to_left_front_caster_wheel: origin xyz=0 0 0 -> xyz=0.375  0.170 0
- joint base_to_left_wheel: origin xyz=0 0 0 -> xyz=0 0.2335 0
- joint base_to_right_back_caster_wheel: origin xyz=0 0 0 -> xyz=-0.375  -0.170 0
- joint base_to_right_front_caster_wheel: origin xyz=0 0 0 -> xyz=0.375  -0.170 0
- joint base_to_right_front_holder: origin xyz=0 0 0 -> xyz=0.4032  -0.170 0.02828
- joint base_to_right_wheel: origin xyz=0 0 0 -> xyz=0 -0.2335 0

Commit message: repositioning
repositioning the right front caster wheel and holder

File: urdf_description/urdf/first.urdf (robot description, URDF)
Before this commit: robot myfirst, 8 links, 7 joints
Joints:
- joint base_to_right_front_caster_wheel: origin xyz=0.375  -0.170 0 -> xyz=0.0565 0 -0.0565
- joint base_to_right_front_holder: origin xyz=0.4032  -0.170 0.02828 -> xyz=0.3749 -0.170 0.0165

Commit message: Adding fix holder
Adding fix holder and making the right caster wheel movable

File: urdf_description/urdf/first.urdf (robot description, URDF)
Before this commit: robot myfirst, 8 links, 7 joints
Links:
- added link right_front_fix_holder; visual box size=0.04 0.04 0.01
Joints:
- removed joint base_to_left_back_caster_wheel
- removed joint base_to_left_front_caster_wheel
- removed joint base_to_left_wheel
- removed joint base_to_right_back_caster_wheel
- removed joint base_to_right_front_caster_wheel
- removed joint base_to_right_front_holder
- removed joint base_to_right_wheel
- added joint joint_left_back_caster_wheel: type fixed, parent base_link, child left_back_caster_wheel, origin xyz=-0.375 0.170 0
- added joint joint_left_front_caster_wheel: type fixed, parent base_link, child left_front_caster_wheel, origin xyz=0.375  0.170 0
- added joint joint_left_wheel: type fixed, parent base_link, child left_wheel, origin xyz=0 0.2335 0
- added joint joint_right_back_caster_wheel: type fixed, parent base_link, child right_back_caster_wheel, origin xyz=-0.375  -0.170 0
- added joint joint_right_front_caster_wheel: type continuous, parent right_front_holder, child right_front_caster_wheel, origin xyz=0.0565 0 -0.0565, axis 0 1 0
- added joint joint_right_front_fix_holder: type fixed, parent base_link, child right_front_fix_holder, origin xyz=0.3749 -0.170 0.0165
- added joint joint_right_front_holder: type continuous, parent right_front_fix_holder, child right_front_holder, origin xyz=0 0 0, axis 0 0 1
- added joint joint_right_wheel: type fixed, parent base_link, child right_wheel, origin xyz=0 -0.2335 0

Commit message: making the right wheel movable
making the right wheel movable

File: urdf_description/urdf/first.urdf (robot description, URDF)
Before this commit: robot myfirst, 9 links, 8 joints
Joints:
- joint joint_right_wheel: axis (none) -> 0 1 0; type fixed -> continuous
