Commit message: update packages

File: my-urdf/my_description/urdf/first.urdf (robot description, URDF)
Before this commit: robot myfirst, 9 links, 8 joints
Links:
- added link left_back_fix_holder; visual box size=0.04 0.04 0.01
- added link left_back_holder; visual box size=0.02 0.08 0.01
- added link left_front_fix_holder; visual box size=0.04 0.04 0.01
- added link left_front_holder; visual box size=0.02 0.08 0.01
- added link right_back_fix_holder; visual box size=0.04 0.04 0.01
- added link right_back_holder; visual box size=0.02 0.08 0.01
Joints:
- added joint joint_left_back_fix_holder: type fixed, parent base_link, child left_back_fix_holder, origin xyz=-0.3749 0.170 0.0165
- added joint joint_left_front_fix_holder: type fixed, parent base_link, child left_front_fix_holder, origin xyz=0.3749 0.170 0.0165
- added joint joint_left_front_holder: type continuous, parent left_front_fix_holder, child left_front_holder, origin xyz=0 0 0, axis 0 0 1
- added joint joint_right_back_fix_holder: type fixed, parent base_link, child right_back_fix_holder, origin xyz=-0.3749 -0.170 0.0165
- added joint left_back_holder: type continuous, parent left_back_fix_holder, child left_back_holder, origin xyz=0 0 0, axis 0 0 1
- added joint right_back_holder: type continuous, parent right_back_fix_holder, child right_back_holder, origin xyz=0 0 0, axis 0 0 1
- joint joint_left_back_caster_wheel: origin xyz=-0.375 0.170 0 -> xyz=-0.0565 0 -0.0565; parent base_link -> left_back_holder
- joint joint_left_front_caster_wheel: origin xyz=0.375  0.170 0 -> xyz=0.0565 0 -0.0565; parent base_link -> left_front_holder
- joint joint_right_back_caster_wheel: origin xyz=-0.375  -0.170 0 -> xyz=-0.0565 0 -0.0565; parent base_link -> right_back_holder

Commit message: adding collision + inertial

File: my-urdf/my_description/urdf/first.urdf (robot description, URDF)
Before this commit: robot myfirst, 15 links, 14 joints
Links:
- link base_link: mass None -> 10; geometry collision box size=1.2 0.6 0.2; visual box size=1.2 0.6 0.2
- link left_back_caster_wheel: mass None -> 0.5; geometry collision cylinder length=0.03 radius=0.04; visual cylinder length=0.03 radius=0.04
- link left_back_fix_holder: mass None -> 0.2; geometry collision box size=0.04 0.04 0.01; visual box size=0.04 0.04 0.01
- link left_back_holder: mass None -> 0.2; geometry collision box size=0.02 0.08 0.01; visual box size=0.02 0.08 0.01
- link left_front_caster_wheel: mass None -> 0.5; geometry collision cylinder length=0.03 radius=0.04; visual cylinder length=0.03 radius=0.04
- link left_front_fix_holder: mass None -> 0.2; geometry collision box size=0.04 0.04 0.01; visual box size=0.04 0.04 0.01
- link left_front_holder: mass None -> 0.2; geometry collision box size=0.02 0.08 0.01; visual box size=0.02 0.08 0.01
- link left_wheel: mass None -> 1; geometry collision cylinder length=0.02 radius=0.08; visual cylinder length=0.02 radius=0.08
- link right_back_caster_wheel: mass None -> 0.5; geometry collision cylinder length=0.03 radius=0.04; visual cylinder length=0.03 radius=0.04
- link right_back_fix_holder: mass None -> 0.2; geometry collision box size=0.04 0.04 0.01; visual box size=0.04 0.04 0.01
- link right_back_holder: mass None -> 0.2; geometry collision box size=0.02 0.08 0.01; visual box size=0.02 0.08 0.01
- link right_front_caster_wheel: mass None -> 0.5; geometry collision cylinder length=0.03 radius=0.04; visual cylinder length=0.03 radius=0.04
- link right_front_fix_holder: mass None -> 0.2; geometry collision box size=0.04 0.04 0.01; visual box size=0.04 0.04 0.01
- link right_front_holder: mass None -> 0.2; geometry collision box size=0.02 0.08 0.01; visual box size=0.02 0.08 0.01
- link right_wheel: mass None -> 1; geometry collision cylinder length=0.02 radius=0.08; visual cylinder length=0.02 radius=0.08
Joints:
- joint joint_left_back_fix_holder: origin xyz=-0.3749 0.170 0.0165 -> xyz=-0.3749 0.170 -0.0335
- joint joint_left_front_fix_holder: origin xyz=0.3749 0.170 0.0165 -> xyz=0.3749 0.170 -0.0335
- joint joint_left_wheel: origin xyz=0 0.2335 0 -> xyz=0 0.2335 -0.05
- joint joint_right_back_fix_holder: origin xyz=-0.3749 -0.170 0.0165 -> xyz=-0.3749 -0.170 -0.0335
- joint joint_right_front_fix_holder: origin xyz=0.3749 -0.170 0.0165 -> xyz=0.3749 -0.170 -0.0335
- joint joint_right_wheel: origin xyz=0 -0.2335 0 -> xyz=0 -0.2335 -0.05

Commit message: adding worlds

File: my-urdf/my_description/urdf/first.urdf (robot description, URDF)
Before this commit: robot myfirst, 15 links, 14 joints
Links:
- added link base_footprint
Joints:
- removed joint joint_left_back_caster_wheel
- removed joint joint_left_back_fix_holder
- removed joint joint_left_front_caster_wheel
- removed joint joint_left_front_fix_holder
- removed joint joint_left_front_holder
- removed joint joint_left_wheel
- removed joint joint_right_back_caster_wheel
- removed joint joint_right_back_fix_holder
- removed joint joint_right_front_caster_wheel
- removed joint joint_right_front_fix_holder
- removed joint joint_right_front_holder
- removed joint joint_right_wheel
- removed joint left_back_holder
- removed joint right_back_holder
- added joint back_holder_right: type continuous, parent right_back_fix_holder, child right_back_holder, origin xyz=0 0 0, axis 0 0 1
- added joint base_link_joint: type fixed, parent base_footprint, child base_link, origin xyz=0 0 0
- added joint left_back_caster_wheel_joint: type continuous, parent left_back_holder, child left_back_caster_wheel, origin xyz=-0.0565 0 -0.0565
- added joint left_back_fix_holder_joint: type fixed, parent base_link, child left_back_fix_holder, origin xyz=-0.3749 0.170 -0.0335
- added joint left_back_holder_joint: type continuous, parent left_back_fix_holder, child left_back_holder, origin xyz=0 0 0, axis 0 0 1
- added joint left_front_caster_wheel_joint: type continuous, parent left_front_holder, child left_front_caster_wheel, origin xyz=0.0565 0 -0.0565, axis 0.0 1.0 0.0
- added joint left_front_fix_holder_joint: type fixed, parent base_link, child left_front_fix_holder, origin xyz=0.3749 0.170 -0.0335
- added joint left_front_holder_joint: type continuous, parent left_front_fix_holder, child left_front_holder, origin xyz=0 0 0, axis 0 0 1
- added joint left_wheel_joint: type continuous, parent base_link, child left_wheel, origin xyz=0 0.2335 -0.05, axis 0.0 1.0 0.0
- added joint right_back_caster_wheel_joint: type continuous, parent right_back_holder, child right_back_caster_wheel, origin xyz=-0.0565 0 -0.0565, axis 0.0 1.0 0.0
- added joint right_back_fix_holder_joint: type fixed, parent base_link, child right_back_fix_holder, origin xyz=-0.3749 -0.170 -0.0335
- added joint right_front_caster_wheel_joint: type continuous, parent right_front_holder, child right_front_caster_wheel, origin xyz=0.0565 0 -0.0565, axis 0 1 0
- added joint right_front_fix_holder_joint: type fixed, parent base_link, child right_front_fix_holder, origin xyz=0.3749 -0.170 -0.0335
- added joint right_front_holder_joint: type continuous, parent right_front_fix_holder, child right_front_holder, origin xyz=0 0 0, axis 0 0 1
- added joint right_wheel_joint: type continuous, parent base_link, child right_wheel, origin xyz=0 -0.2335 -0.05, axis 0 1 0
